Commit message: add: scan_bot running

File: spcbot_description/urdf/scanner_bot.gazebo.xacro (robot description, xacro)
@@ -1,71 +1,5 @@
 <?xml version='1.0'?>
-<robot name="spcbot_gazebo" xmlns:xacro="http://ros.org/wiki/xacro">
-  <!-- Camera Plugin -->
-  <gazebo reference="camera_link">
-    <material>Gazebo/Green</material>
-    <sensor type="camera" name="camera">
-      <update_rate>30.0</update_rate>
-      <visualize></visualize>
-      <camera name="head">
-        <horizontal_fov>1.3962634</horizontal_fov>
-        <image>
-          <width>800</width>
-          <height>800</height>
-          <format>R8G8B8</format>
-        </image>
-        <clip>
-          <near>0.02</near>
-          <far>300</far>
-        </clip>
-      </camera>
-      <plugin name="camera_controller" filename="libgazebo_ros_camera.so">
-        <alwaysOn>true</alwaysOn>
-        <updateRate>0.0</updateRate>
-        <cameraName>spcbot/camera</cameraName>
-        <imageTopicName>image_raw</imageTopicName>
-        <cameraInfoTopicName>camera_info</cameraInfoTopicName>
-        <frameName>camera</frameName>
-        <hackBaseline>0.07</hackBaseline>
-        <distortionK1>0.0</distortionK1>
-        <distortionK2>0.0</distortionK2>
-        <distortionK3>0.0</distortionK3>
-        <distortionT1>0.0</distortionT1>
-        <distortionT2>0.0</distortionT2>
-      </plugin>
-    </sensor>
-  </gazebo>
-  <!-- Whells Plugin -->
-  <gazebo>
-    <plugin name="differential_drive_controller" filename="libgazebo_ros_diff_drive.so">
-      <legacyMode>false</legacyMode>
-      <alwaysOn>true</alwaysOn>
-      <updateRate>10</updateRate>
-      <leftJoint>left_wheel_hinge</leftJoint>
-      <rightJoint>right_wheel_hinge</rightJoint>
-      <wheelSeparation>0.30</wheelSeparation>
-      <wheelDiameter>0.2</wheelDiameter>
-      <torque>30</torque>
-      <commandTopic>cmd_vel</commandTopic>
-      <odometryTopic>odom</odometryTopic>
-      <odometryFrame>odom</odometryFrame>
-      <robotBaseFrame>chassis</robotBaseFrame>
-    </plugin>
-  </gazebo>
-  <gazebo reference="chassis">
-      <material>
-        Gazebo/Black
-      </material>
-  </gazebo>
-  <gazebo reference="left_wheel">
-      <material>
-        Gazebo/Yellow
-      </material>
-  </gazebo>
-  <gazebo reference="right_wheel">
-      <material>
-        Gazebo/Yellow
-      </material>
-  </gazebo>
-<!-- 2D LiDAR Plugin -->
+<robot name="scanner_bot_gazebo" xmlns:xacro="http://ros.org/wiki/xacro">
+    <!-- 2D LiDAR Plugin -->
   <gazebo reference="hokuyo_link">
     <sensor type="ray" name="head_hokuyo_sensor">

File: spcbot_description/urdf/spcbot.urdf.xacro (robot description, xacro)
@@ -139,4 +139,5 @@
     <joint_properties damping="0.0" friction="0.0"/>
   </joint>
+  <!-- Camera -->
   <link name="camera_link">
     <collision>
